File: mcu.sch (KiCad schematic (older format))
At the start: 68 parts, among them J10 JTAG, J11 esp32L, J12 esp32B, J13 esp32R, J2 SPI1, J3 uSD, J4 I2C1, J5 serial1, J6 serial2, J7 touch interface, J8 LCD 4.3, J9 EXT_IOS, SW1 reset, U3 AT25SF641, U5 STM32F750Z8, U6 MP3302DJ-LF-P, U7 ESP32-WROOM-32, U8 ASDMB-25.000MHZ-LC-T, Y2 32.768 kHz

Commit message: nope
Parts:
- removed C29: 100nF, symbol Device:C_Small
- removed R25: 10k, symbol Device:R_Small
- removed R26: 100, symbol Device:R_Small
- removed U8: ASDMB-25.000MHZ-LC-T, Oscillator:Oscillator_SMD_Abracon_ASDMB-4Pin_2.5x2.0mm, symbol Oscillator:ASDMB-xxxMHz
- added C? (x2): 22pF, symbol Device:C_Small
- added Y?: 25MHz, symbol Device:Crystal
Connections:
- net GND: now also C?.2, C?.2
- net at U5.23 (PH0): now also C?.1, Y?.2
- net at U5.24 (PH1): now also C?.1, Y?.1
- no-connect marks 16 -> 15
Changed lines of the file:
@@
 Text GLabel 12750 8550 0    39   Input ~ 0
 EXTIO_3
-$Comp
-L d_st:STM32F750Z8 U5
-U 1 1 5F863DEB
-P 13900 2050
-F 0 "U5" H 13900 -500 157 0000 C CNN
-F 1 "STM32F750Z8" H 13900 3250 157 0000 C CNN
-F 2 "" H 13800 2200 157 0001 C CNN
-F 3 "" H 13800 2200 157 0001 C CNN
-	1    13900 2050
-	1    0    0    -1
-$EndComp
 Text Notes 14600 2900 0    39   ~ 0
 input
@@
 Wire Wire Line
 	10600 1850 10900 1850
-Text Notes 11550 4200 0    39   ~ 0
+Text Notes 11650 4100 0    39   ~ 0
 validate caps against\nchoosen xtal
 $Comp
@@
 ABS07-166-32.768KHZ-T
 $Comp
-L Oscillator:ASDMB-xxxMHz U8
-U 1 1 60FEB22A
-P 10600 2950
-F 0 "U8" H 11044 2996 50  0000 L CNN
-F 1 "ASDMB-25.000MHZ-LC-T" H 10100 2500 50  0000 L CNN
-F 2 "Oscillator:Oscillator_SMD_Abracon_ASDMB-4Pin_2.5x2.0mm" H 10600 2950 50  0001 C CNN
-F 3 "https://abracon.com/Oscillators/ASDMB.pdf" H 10900 3400 50  0001 C CNN
-	1    10600 2950
-	1    0    0    -1
-$EndComp
-$Comp
-L Device:R_Small R25
-U 1 1 60FEC7BE
-P 10000 2950
-F 0 "R25" V 10196 2950 50  0000 C CNN
-F 1 "10k" V 10105 2950 50  0000 C CNN
-F 2 "" H 10000 2950 50  0001 C CNN
-F 3 "~" H 10000 2950 50  0001 C CNN
-	1    10000 2950
+L d_st:STM32F750Z8 U5
+U 1 1 5F863DEB
+P 13900 2050
+F 0 "U5" H 13900 -500 157 0000 C CNN
+F 1 "STM32F750Z8" H 13900 3250 157 0000 C CNN
+F 2 "" H 13800 2200 157 0001 C CNN
+F 3 "" H 13800 2200 157 0001 C CNN
+	1    13900 2050
+	1    0    0    -1
+$EndComp
+$Comp
+L Device:Crystal Y?
+U 1 1 6102B495
+P 12150 3600
+F 0 "Y?" V 12196 3469 50  0000 R CNN
+F 1 "25MHz" V 12105 3469 50  0000 R CNN
+F 2 "" H 12150 3600 50  0001 C CNN
+F 3 "~" H 12150 3600 50  0001 C CNN
+	1    12150 3600
 	0    -1   -1   0
 $EndComp
 $Comp
-L Device:C_Small C29
-U 1 1 60FED86D
-P 9850 3150
-F 0 "C29" H 9942 3196 50  0000 L CNN
-F 1 "100nF" H 9942 3105 50  0000 L CNN
-F 2 "" H 9850 3150 50  0001 C CNN
-F 3 "~" H 9850 3150 50  0001 C CNN
-	1    9850 3150
-	1    0    0    -1
-$EndComp
-$Comp
-L power:+3.3V #PWR045
-U 1 1 60FEF86B
-P 9850 2650
-F 0 "#PWR045" H 9850 2500 50  0001 C CNN
-F 1 "+3.3V" H 9865 2823 50  0000 C CNN
-F 2 "" H 9850 2650 50  0001 C CNN
-F 3 "" H 9850 2650 50  0001 C CNN
-	1    9850 2650
-	1    0    0    -1
-$EndComp
-$Comp
-L power:GND #PWR046
-U 1 1 60FEFF10
-P 9850 3250
-F 0 "#PWR046" H 9850 3000 50  0001 C CNN
-F 1 "GND" H 9855 3077 50  0000 C CNN
-F 2 "" H 9850 3250 50  0001 C CNN
-F 3 "" H 9850 3250 50  0001 C CNN
-	1    9850 3250
-	1    0    0    -1
-$EndComp
-Wire Wire Line
-	10700 3250 9850 3250
-Connection ~ 9850 3250
-Wire Wire Line
-	9850 3050 9850 2950
-Wire Wire Line
-	9900 2950 9850 2950
-Connection ~ 9850 2950
-Wire Wire Line
-	9850 2950 9850 2650
-Wire Wire Line
-	10700 2650 9850 2650
-Connection ~ 9850 2650
-Wire Wire Line
-	10100 2950 10200 2950
-$Comp
-L Device:R_Small R26
-U 1 1 61011743
-P 12200 3550
-F 0 "R26" V 12004 3550 50  0000 C CNN
-F 1 "100" V 12095 3550 50  0000 C CNN
-F 2 "" H 12200 3550 50  0001 C CNN
-F 3 "~" H 12200 3550 50  0001 C CNN
-	1    12200 3550
-	0    1    1    0
-$EndComp
-Wire Wire Line
-	12300 3550 12750 3550
-Wire Wire Line
-	12100 3550 11650 3550
-Wire Wire Line
-	11650 3550 11650 2950
-Wire Wire Line
-	11650 2950 11000 2950
-Text Label 11250 2950 0    39   ~ 0
-OSC_25M
-NoConn ~ 12750 3650
+L Device:C_Small C?
+U 1 1 6102D7D8
+P 11850 3450
+F 0 "C?" V 11621 3450 50  0000 C CNN
+F 1 "22pF" V 11712 3450 50  0000 C CNN
+F 2 "" H 11850 3450 50  0001 C CNN
+F 3 "~" H 11850 3450 50  0001 C CNN
+	1    11850 3450
+	0    1    1    0
+$EndComp
+$Comp
+L Device:C_Small C?
+U 1 1 6102DD67
+P 11850 3750
+F 0 "C?" V 12050 3750 50  0000 C CNN
+F 1 "22pF" V 11950 3750 50  0000 C CNN
+F 2 "" H 11850 3750 50  0001 C CNN
+F 3 "~" H 11850 3750 50  0001 C CNN
+	1    11850 3750
+	0    1    1    0
+$EndComp
+$Comp
+L power:GND #PWR?
+U 1 1 6102E30B
+P 11600 3450
+F 0 "#PWR?" H 11600 3200 50  0001 C CNN
+F 1 "GND" H 11605 3277 50  0000 C CNN
+F 2 "" H 11600 3450 50  0001 C CNN
+F 3 "" H 11600 3450 50  0001 C CNN
+	1    11600 3450
+	0    1    1    0
+$EndComp
+Wire Wire Line
+	11600 3450 11700 3450
+Wire Wire Line
+	11700 3450 11700 3750
+Wire Wire Line
+	11700 3750 11750 3750
+Connection ~ 11700 3450
+Wire Wire Line
+	11700 3450 11750 3450
+Wire Wire Line
+	11950 3450 12150 3450
+Wire Wire Line
+	12600 3450 12600 3550
+Wire Wire Line
+	12600 3550 12750 3550
+Wire Wire Line
+	12750 3650 12600 3650
+Wire Wire Line
+	12600 3650 12600 3750
+Wire Wire Line
+	12600 3750 12150 3750
+Connection ~ 12150 3750
+Wire Wire Line
+	12150 3750 11950 3750
+Connection ~ 12150 3450
+Wire Wire Line
+	12150 3450 12600 3450
 $EndSCHEMATC
