File: mcu.sch (KiCad schematic (older format))
At the start: 67 parts, among them J10 JTAG, J11 esp32L, J12 esp32B, J13 esp32R, J2 SPI1, J3 uSD, J4 I2C1, J5 serial1, J6 serial2, J7 touch interface, J8 LCD 4.3, J9 EXT_IOS, SW1 reset, U3 AT25SF641, U5 STM32F750Z8, U6 MP3302DJ-LF-P, U7 ESP32-WROOM-32, Y2 32.768 kHz

Commit message: good one
Parts:
- removed Y?: 25MHz, symbol Device:Crystal
- added R25: 0, symbol Device:R_Small
- added Y1: 25MHz, symbol Device:Crystal_GND24_Small
- C29, C30: renamed from C?; value 22pF -> 16pF
Connections:
- wire segments 134 -> 135
Other:
- note added: "ABMM2-25.000MHZ-D1-T\nLc=18pF\nCstray=10pF\nCl=(16*16)/(16+16)+10"
- note removed: "validate caps against\nchoosen xtal"
Changed lines of the file:
@@
 Wire Wire Line
 	10600 1850 10900 1850
-Text Notes 11650 4100 0    39   ~ 0
-validate caps against\nchoosen xtal
 $Comp
 L power:+3.3V #PWR0142
@@
 $EndComp
 $Comp
-L Device:Crystal Y?
-U 1 1 6102B495
-P 12150 3600
-F 0 "Y?" V 12196 3469 50  0000 R CNN
-F 1 "25MHz" V 12105 3469 50  0000 R CNN
-F 2 "" H 12150 3600 50  0001 C CNN
-F 3 "~" H 12150 3600 50  0001 C CNN
-	1    12150 3600
-	0    -1   -1   0
-$EndComp
-$Comp
-L Device:C_Small C?
+L Device:C_Small C29
 U 1 1 6102D7D8
 P 11850 3450
-F 0 "C?" V 11621 3450 50  0000 C CNN
-F 1 "22pF" V 11712 3450 50  0000 C CNN
+F 0 "C29" V 11621 3450 50  0000 C CNN
+F 1 "16pF" V 11712 3450 50  0000 C CNN
 F 2 "" H 11850 3450 50  0001 C CNN
 F 3 "~" H 11850 3450 50  0001 C CNN
@@
 $EndComp
 $Comp
-L Device:C_Small C?
+L Device:C_Small C30
 U 1 1 6102DD67
 P 11850 3750
-F 0 "C?" V 12050 3750 50  0000 C CNN
-F 1 "22pF" V 11950 3750 50  0000 C CNN
+F 0 "C30" V 12050 3750 50  0000 C CNN
+F 1 "16pF" V 11950 3750 50  0000 C CNN
 F 2 "" H 11850 3750 50  0001 C CNN
 F 3 "~" H 11850 3750 50  0001 C CNN
@@
 $EndComp
 $Comp
-L power:GND #PWR?
+L power:GND #PWR045
 U 1 1 6102E30B
 P 11600 3450
-F 0 "#PWR?" H 11600 3200 50  0001 C CNN
+F 0 "#PWR045" H 11600 3200 50  0001 C CNN
 F 1 "GND" H 11605 3277 50  0000 C CNN
 F 2 "" H 11600 3450 50  0001 C CNN
@@
 	11700 3450 11750 3450
 Wire Wire Line
+	12600 3450 12600 3550
+Wire Wire Line
+	12600 3550 12750 3550
+Wire Wire Line
+	11950 3750 12150 3750
+Wire Wire Line
 	11950 3450 12150 3450
-Wire Wire Line
-	12600 3450 12600 3550
-Wire Wire Line
-	12600 3550 12750 3550
-Wire Wire Line
-	12750 3650 12600 3650
-Wire Wire Line
-	12600 3650 12600 3750
-Wire Wire Line
-	12600 3750 12150 3750
+$Comp
+L Device:Crystal_GND24_Small Y1
+U 1 1 6105E2FC
+P 12150 3600
+F 0 "Y1" V 12050 3650 50  0000 L CNN
+F 1 "25MHz" V 12250 3650 50  0000 L CNN
+F 2 "" H 12150 3600 50  0001 C CNN
+F 3 "~" H 12150 3600 50  0001 C CNN
+F 4 "815-ABMM2-25-D1T" V 12150 3600 50  0001 C CNN "mouser"
+	1    12150 3600
+	0    1    1    0
+$EndComp
+Wire Wire Line
+	12150 3500 12150 3450
+Connection ~ 12150 3450
+Wire Wire Line
+	12150 3450 12600 3450
+Wire Wire Line
+	12150 3700 12150 3750
+$Comp
+L power:GND #PWR046
+U 1 1 6106B18B
+P 12050 3600
+F 0 "#PWR046" H 12050 3350 50  0001 C CNN
+F 1 "GND" H 12055 3427 50  0000 C CNN
+F 2 "" H 12050 3600 50  0001 C CNN
+F 3 "" H 12050 3600 50  0001 C CNN
+	1    12050 3600
+	0    1    1    0
+$EndComp
+$Comp
+L power:GND #PWR047
+U 1 1 6106B489
+P 12250 3600
+F 0 "#PWR047" H 12250 3350 50  0001 C CNN
+F 1 "GND" H 12255 3427 50  0000 C CNN
+F 2 "" H 12250 3600 50  0001 C CNN
+F 3 "" H 12250 3600 50  0001 C CNN
+	1    12250 3600
+	0    -1   -1   0
+$EndComp
+$Comp
+L Device:R_Small R25
+U 1 1 6106D61B
+P 12650 3650
+F 0 "R25" V 12454 3650 50  0000 C CNN
+F 1 "0" V 12545 3650 50  0000 C CNN
+F 2 "" H 12650 3650 50  0001 C CNN
+F 3 "~" H 12650 3650 50  0001 C CNN
+	1    12650 3650
+	0    1    1    0
+$EndComp
+Wire Wire Line
+	12550 3650 12550 3750
+Wire Wire Line
+	12550 3750 12150 3750
 Connection ~ 12150 3750
-Wire Wire Line
-	12150 3750 11950 3750
-Connection ~ 12150 3450
-Wire Wire Line
-	12150 3450 12600 3450
+Text Notes 11950 3400 0    39   ~ 0
+ABMM2-25.000MHZ-D1-T\nLc=18pF\nCstray=10pF\nCl=(16*16)/(16+16)+10
 $EndSCHEMATC

Commit message: squeak
Parts:
- removed JP2: serTX, symbol Device:Jumper_NC_Small
- removed JP3: serRX, symbol Device:Jumper_NC_Small
- added JP2: esp32 tx src, symbol Jumper:Jumper_3_Bridged12
- added JP3: esp32 rx src, symbol Jumper:Jumper_3_Bridged12
Connections:
- net labels added: ESP32_RX_SRC, ESP32_TX_SRC
- wire segments 135 -> 133
Changed lines of the file:
@@
 Text Notes 13100 8300 0    39   ~ 0
 keyboard col in
-Text GLabel 2900 1700 2    39   Input ~ 0
-SERIAL3_RX
-Text GLabel 3000 1500 2    39   Input ~ 0
-SERIAL3_TX
 Text GLabel 12750 4750 0    39   Input ~ 0
 SERIAL3_RX
@@
 $EndComp
 Wire Wire Line
-	2900 1700 2800 1700
-Wire Wire Line
-	3000 1500 2800 1500
-Wire Wire Line
 	8100 5500 8050 5500
 Connection ~ 8050 5500
@@
 Text GLabel 1600 1700 0    39   Input ~ 0
 esp32_sens_vn
-$Comp
-L Device:Jumper_NC_Small JP2
-U 1 1 60FA4DA3
-P 4000 3100
-F 0 "JP2" H 4000 3312 50  0000 C CNN
-F 1 "serTX" H 4000 3221 50  0000 C CNN
-F 2 "" H 4000 3100 50  0001 C CNN
-F 3 "~" H 4000 3100 50  0001 C CNN
-	1    4000 3100
-	1    0    0    -1
-$EndComp
-$Comp
-L Device:Jumper_NC_Small JP3
-U 1 1 60FA5BE1
-P 4000 3400
-F 0 "JP3" H 4000 3612 50  0000 C CNN
-F 1 "serRX" H 4000 3521 50  0000 C CNN
-F 2 "" H 4000 3400 50  0001 C CNN
-F 3 "~" H 4000 3400 50  0001 C CNN
-	1    4000 3400
-	1    0    0    -1
-$EndComp
-Text GLabel 3900 3100 0    39   Input ~ 0
+Text GLabel 4000 3900 0    39   Input ~ 0
 SERIAL3_TX
-Text GLabel 3900 3400 0    39   Input ~ 0
+Text GLabel 4000 4550 0    39   Input ~ 0
 SERIAL3_RX
-Text GLabel 4100 3100 2    39   Input ~ 0
+Text GLabel 4500 3900 2    39   Input ~ 0
 esp32_iotxd0
-Text GLabel 4100 3400 2    39   Input ~ 0
+Text GLabel 4500 4550 2    39   Input ~ 0
 esp32_iorxd0
 Text GLabel 2800 3600 2    39   Input ~ 0
@@
 Text Notes 11950 3400 0    39   ~ 0
 ABMM2-25.000MHZ-D1-T\nLc=18pF\nCstray=10pF\nCl=(16*16)/(16+16)+10
+$Comp
+L Jumper:Jumper_3_Bridged12 JP2
+U 1 1 6107F2AD
+P 4250 3900
+F 0 "JP2" H 4250 4104 50  0000 C CNN
+F 1 "esp32 tx src" H 4250 4013 50  0000 C CNN
+F 2 "" H 4250 3900 50  0001 C CNN
+F 3 "~" H 4250 3900 50  0001 C CNN
+	1    4250 3900
+	1    0    0    -1
+$EndComp
+$Comp
+L Jumper:Jumper_3_Bridged12 JP3
+U 1 1 6107F61A
+P 4250 4550
+F 0 "JP3" H 4250 4754 50  0000 C CNN
+F 1 "esp32 rx src" H 4250 4663 50  0000 C CNN
+F 2 "" H 4250 4550 50  0001 C CNN
+F 3 "~" H 4250 4550 50  0001 C CNN
+	1    4250 4550
+	1    0    0    -1
+$EndComp
+Text GLabel 2800 1500 2    39   Input ~ 0
+ESP32_TX_SRC
+Text GLabel 4250 4050 2    39   Input ~ 0
+ESP32_TX_SRC
+Text GLabel 2800 1700 2    39   Input ~ 0
+ESP32_RX_SRC
+Text GLabel 4250 4700 2    39   Input ~ 0
+ESP32_RX_SRC
 $EndSCHEMATC

Commit message: Use libs; start assigning footprints
Parts:
- D5: footprint (none) -> Diode_SMD:D_SMB_Handsoldering
- U5: footprint (none) -> Package_QFP:LQFP-144_20x20mm_P0.5mm
- U6: footprint IC5_MP3302DJ-LF-P_MNP -> d_mps:MP3302DJ-LF-P
- Y1: footprint (none) -> Crystal:Crystal_SMD_0603-4Pin_6.0x3.5mm_HandSoldering
- Y2: footprint (none) -> Crystal:Crystal_SMD_G8-2Pin_3.2x1.5mm_HandSoldering
Changed lines of the file:
@@
 F 0 "Y2" H 15950 7268 50  0000 C CNN
 F 1 "32.768 kHz" H 15950 7177 50  0000 C CNN
-F 2 "" H 15950 7000 50  0001 C CNN
+F 2 "Crystal:Crystal_SMD_G8-2Pin_3.2x1.5mm_HandSoldering" H 15950 7000 50  0001 C CNN
 F 3 "~" H 15950 7000 50  0001 C CNN
 F 4 "815-ABS0716632.768KT" H 15950 7000 50  0001 C CNN "mouser"
@@
 F 0 "U6" H 8850 6387 60  0000 C CNN
 F 1 "MP3302DJ-LF-P" H 8850 6281 60  0000 C CNN
-F 2 "IC5_MP3302DJ-LF-P_MNP" H 8850 6240 60  0001 C CNN
+F 2 "d_mps:MP3302DJ-LF-P" H 8850 6240 60  0001 C CNN
 F 3 "" H 8050 6000 60  0000 C CNN
 	1    8050 6000
@@
 F 0 "D5" H 8250 5283 50  0000 C CNN
 F 1 "MBRS140T3G" H 8250 5374 50  0000 C CNN
-F 2 "" H 8250 5500 50  0001 C CNN
+F 2 "Diode_SMD:D_SMB_Handsoldering" H 8250 5500 50  0001 C CNN
 F 3 "~" H 8250 5500 50  0001 C CNN
 	1    8250 5500
@@
 F 0 "U5" H 13900 -500 157 0000 C CNN
 F 1 "STM32F750Z8" H 13900 3250 157 0000 C CNN
-F 2 "" H 13800 2200 157 0001 C CNN
+F 2 "Package_QFP:LQFP-144_20x20mm_P0.5mm" H 13800 2200 157 0001 C CNN
 F 3 "" H 13800 2200 157 0001 C CNN
 	1    13900 2050
@@
 F 0 "Y1" V 12050 3650 50  0000 L CNN
 F 1 "25MHz" V 12250 3650 50  0000 L CNN
-F 2 "" H 12150 3600 50  0001 C CNN
+F 2 "Crystal:Crystal_SMD_0603-4Pin_6.0x3.5mm_HandSoldering" H 12150 3600 50  0001 C CNN
 F 3 "~" H 12150 3600 50  0001 C CNN
 F 4 "815-ABMM2-25-D1T" V 12150 3600 50  0001 C CNN "mouser"

Commit message: Assigning footprints
Parts:
- BZ1: footprint (none) -> Buzzer_Beeper:Buzzer_Murata_PKMCS0909E4000-R1
- C10, C14, C27, C28, C29, C3, C30, C31, C32, C33, C34, C35, C36, C37, C38, C39: footprint (none) -> Capacitor_SMD:C_0805_2012Metric_Pad1.18x1.45mm_HandSolder
- D4: mouser (none) -> 859-LTST-S310F2KT
- J10: footprint (none) -> Connector_PinHeader_2.54mm:PinHeader_2x05_P2.54mm_Vertical
- J11, J13: footprint (none) -> Connector_PinSocket_1.27mm:PinSocket_1x14_P1.27mm_Vertical
- J12: footprint (none) -> Connector_PinSocket_1.27mm:PinSocket_1x10_P1.27mm_Vertical
- J2, J9: footprint (none) -> Connector_PinHeader_2.54mm:PinHeader_1x06_P2.54mm_Horizontal
- J3: footprint (none) -> Connector_Card:microSD_HC_Wuerth_693072010801
- J4: footprint (none) -> Connector_PinHeader_2.54mm:PinHeader_1x05_P2.54mm_Horizontal
- J5, J6: footprint (none) -> Connector_PinHeader_2.54mm:PinHeader_1x03_P2.54mm_Horizontal
- J7: footprint (none) -> Connector_FFC-FPC:TE_0-1734839-8_1x08-1MP_P0.5mm_Horizontal
- J8: footprint (none) -> Connector_FFC-FPC:TE_4-1734839-0_1x40-1MP_P0.5mm_Horizontal
- JP2, JP3: footprint (none) -> Jumper:SolderJumper-3_P1.3mm_Bridged2Bar12_Pad1.0x1.5mm_NumberLabels
- L2: footprint (none) -> Inductor_SMD:L_0805_2012Metric_Pad1.05x1.20mm_HandSolder; mouser (none) -> 963-LBR2012T220K
- R10, R11, R12, R16, R17, R18, R19, R2, R20, R21, R22, R23, R24, R25, R3, R4, R5, R7, R8, R9: footprint (none) -> Resistor_SMD:R_0805_2012Metric_Pad1.20x1.40mm_HandSolder
- SW1: footprint (none) -> Button_Switch_SMD:SW_SPST_EVQQ2
- TP1, TP2, TP3, TP4, TP5, TP6, TP7: footprint (none) -> TestPoint:TestPoint_Keystone_5010-5014_Multipurpose

Commit message: more assign; rework rgb led
Parts:
- added Q1, Q2, Q3: ZXMN2F30FH, Package_TO_SOT_SMD:SOT-23, symbol Transistor_FET:ZXMN2F30FH
- D4: symbol Device:LED_GCBR -> Device:LED_GABR
- R3, R4: value 220 -> 56
- R5: value 220 -> 100
Connections:
- net +3V3: now also D4.2 (A)
- net GND: now also Q1.2 (S), Q2.2 (S), Q3.2 (S); no longer D4.2 (K)
- net RGBLED1_B: now also Q1.1 (G); no longer R5.1
- net RGBLED1_G: now also Q2.1 (G); no longer R4.1
- net RGBLED1_R: now also Q3.1 (G); no longer R3.1
- net at D4.3 (BK): now also R3.2; no longer R5.2
- net at D4.4 (RK): now also R5.2; no longer R3.2
- new net: Q3.3 (D), R5.1
- new net: Q2.3 (D), R4.1
- new net: Q1.3 (D), R3.1
Other:
- note added: "pull down each"
- moved on the sheet: D4
Changed lines of the file:
@@
 $EndComp
 $Comp
-L Device:LED_GCBR D4
+L Device:LED_GABR D4
 U 1 1 5F871F9B
-P 11050 9600
-F 0 "D4" H 11050 10097 50  0000 C CNN
-F 1 "LED_GCBR_1" H 11050 10006 50  0000 C CNN
-F 2 "" H 11050 9550 50  0001 C CNN
-F 3 "~" H 11050 9550 50  0001 C CNN
-F 4 "859-LTST-S310F2KT" H 11050 9600 50  0001 C CNN "mouser"
-	1    11050 9600
-	1    0    0    -1
-$EndComp
-Text GLabel 11450 9400 2    50   Input ~ 0
+P 9900 10300
+F 0 "D4" H 9900 10797 50  0000 C CNN
+F 1 "LED_GCBR_1" H 9900 10706 50  0000 C CNN
+F 2 "" H 9900 10250 50  0001 C CNN
+F 3 "~" H 9900 10250 50  0001 C CNN
+F 4 "859-LTST-S310F2KT" H 9900 10300 50  0001 C CNN "mouser"
+	1    9900 10300
+	-1   0    0    1
+$EndComp
+Text GLabel 11550 9600 2    50   Input ~ 0
 RGBLED1_R
-Text GLabel 11450 9600 2    50   Input ~ 0
+Text GLabel 11050 9600 2    50   Input ~ 0
 RGBLED1_G
-Text GLabel 11450 9800 2    50   Input ~ 0
+Text GLabel 10550 9600 2    50   Input ~ 0
 RGBLED1_B
-$Comp
-L power:GND #PWR025
-U 1 1 5F88DB4B
-P 10850 9600
-F 0 "#PWR025" H 10850 9350 50  0001 C CNN
-F 1 "GND" V 10855 9472 50  0000 R CNN
-F 2 "" H 10850 9600 50  0001 C CNN
-F 3 "" H 10850 9600 50  0001 C CNN
-	1    10850 9600
-	0    1    1    0
-$EndComp
-$Comp
-L Device:R_Small R3
-U 1 1 5F895090
-P 11350 9400
-F 0 "R3" V 11250 9400 50  0000 C CNN
-F 1 "220" V 11350 9400 50  0000 C CNN
-F 2 "Resistor_SMD:R_0805_2012Metric_Pad1.20x1.40mm_HandSolder" H 11350 9400 50  0001 C CNN
-F 3 "~" H 11350 9400 50  0001 C CNN
-	1    11350 9400
-	0    1    1    0
-$EndComp
-$Comp
-L Device:R_Small R4
-U 1 1 5F8957F6
-P 11350 9600
-F 0 "R4" V 11250 9600 50  0000 C CNN
-F 1 "220" V 11350 9600 50  0000 C CNN
-F 2 "Resistor_SMD:R_0805_2012Metric_Pad1.20x1.40mm_HandSolder" H 11350 9600 50  0001 C CNN
-F 3 "~" H 11350 9600 50  0001 C CNN
-	1    11350 9600
-	0    1    1    0
-$EndComp
-$Comp
-L Device:R_Small R5
-U 1 1 5F895B83
-P 11350 9800
-F 0 "R5" V 11250 9800 50  0000 C CNN
-F 1 "220" V 11350 9800 50  0000 C CNN
-F 2 "Resistor_SMD:R_0805_2012Metric_Pad1.20x1.40mm_HandSolder" H 11350 9800 50  0001 C CNN
-F 3 "~" H 11350 9800 50  0001 C CNN
-	1    11350 9800
-	0    1    1    0
-$EndComp
 Text GLabel 15050 7650 2    50   Input ~ 0
 RGBLED1_R
@@
 Wire Notes Line
 	3850 5000 3850 8450
-Text Notes 10550 9000 0    118  ~ 0
+Text Notes 10600 9200 0    118  ~ 0
 RGB Led status
 Text Notes 8300 8250 0    118  ~ 0
@@
 Wire Notes Line
 	12200 7950 12200 9950
-Wire Notes Line
-	500  9950 12200 9950
 Wire Notes Line
 	7050 7950 12200 7950
@@
 Text GLabel 4250 4700 2    39   Input ~ 0
 ESP32_RX_SRC
+$Comp
+L Transistor_FET:ZXMN2F30FH Q3
+U 1 1 61189A26
+P 11550 9800
+F 0 "Q3" H 11754 9846 50  0000 L CNN
+F 1 "ZXMN2F30FH" H 11754 9755 50  0000 L CNN
+F 2 "Package_TO_SOT_SMD:SOT-23" H 11750 9725 50  0001 L CIN
+F 3 "http://www.diodes.com/assets/Datasheets/ZXMN2F30FH.pdf" H 11550 9800 50  0001 L CNN
+F 4 "522-ZXMN2F30FHTA" H 11550 9800 50  0001 C CNN "mouser"
+	1    11550 9800
+	0    1    1    0
+$EndComp
+$Comp
+L Transistor_FET:ZXMN2F30FH Q2
+U 1 1 6118D033
+P 11050 9800
+F 0 "Q2" H 11254 9846 50  0000 L CNN
+F 1 "ZXMN2F30FH" H 11254 9755 50  0000 L CNN
+F 2 "Package_TO_SOT_SMD:SOT-23" H 11250 9725 50  0001 L CIN
+F 3 "http://www.diodes.com/assets/Datasheets/ZXMN2F30FH.pdf" H 11050 9800 50  0001 L CNN
+F 4 "522-ZXMN2F30FHTA" H 11050 9800 50  0001 C CNN "mouser"
+	1    11050 9800
+	0    1    1    0
+$EndComp
+Wire Notes Line
+	10250 9950 500  9950
+$Comp
+L Transistor_FET:ZXMN2F30FH Q1
+U 1 1 611A743F
+P 10550 9800
+F 0 "Q1" H 10754 9846 50  0000 L CNN
+F 1 "ZXMN2F30FH" H 10754 9755 50  0000 L CNN
+F 2 "Package_TO_SOT_SMD:SOT-23" H 10750 9725 50  0001 L CIN
+F 3 "http://www.diodes.com/assets/Datasheets/ZXMN2F30FH.pdf" H 10550 9800 50  0001 L CNN
+F 4 "522-ZXMN2F30FHTA" H 10550 9800 50  0001 C CNN "mouser"
+	1    10550 9800
+	0    1    1    0
+$EndComp
+Text Notes 11450 9489 2    39   ~ 0
+pull down each
+$Comp
+L power:GND #PWR0102
+U 1 1 611D3B05
+P 11350 9900
+F 0 "#PWR0102" H 11350 9650 50  0001 C CNN
+F 1 "GND" V 11355 9772 50  0000 R CNN
+F 2 "" H 11350 9900 50  0001 C CNN
+F 3 "" H 11350 9900 50  0001 C CNN
+	1    11350 9900
+	-1   0    0    1
+$EndComp
+$Comp
+L power:GND #PWR0104
+U 1 1 611D4194
+P 10850 9900
+F 0 "#PWR0104" H 10850 9650 50  0001 C CNN
+F 1 "GND" V 10855 9772 50  0000 R CNN
+F 2 "" H 10850 9900 50  0001 C CNN
+F 3 "" H 10850 9900 50  0001 C CNN
+	1    10850 9900
+	-1   0    0    1
+$EndComp
+$Comp
+L power:GND #PWR0105
+U 1 1 611D45A9
+P 10350 9900
+F 0 "#PWR0105" H 10350 9650 50  0001 C CNN
+F 1 "GND" V 10355 9772 50  0000 R CNN
+F 2 "" H 10350 9900 50  0001 C CNN
+F 3 "" H 10350 9900 50  0001 C CNN
+	1    10350 9900
+	-1   0    0    1
+$EndComp
+Wire Wire Line
+	10750 10100 10750 9900
+Wire Wire Line
+	11250 9900 11250 10300
+Wire Wire Line
+	11750 10500 11750 9900
+$Comp
+L power:+3.3V #PWR0110
+U 1 1 611EBD7D
+P 9700 10300
+F 0 "#PWR0110" H 9700 10150 50  0001 C CNN
+F 1 "+3.3V" H 9715 10473 50  0000 C CNN
+F 2 "" H 9700 10300 50  0001 C CNN
+F 3 "" H 9700 10300 50  0001 C CNN
+	1    9700 10300
+	0    -1   -1   0
+$EndComp
+Wire Notes Line
+	9350 9950 9350 11200
+$Comp
+L Device:R_Small R3
+U 1 1 612250FD
+P 10200 10100
+F 0 "R3" V 10004 10100 50  0000 C CNN
+F 1 "56" V 10095 10100 50  0000 C CNN
+F 2 "Resistor_SMD:R_0805_2012Metric_Pad1.20x1.40mm_HandSolder" H 10200 10100 50  0001 C CNN
+F 3 "~" H 10200 10100 50  0001 C CNN
+	1    10200 10100
+	0    1    1    0
+$EndComp
+$Comp
+L Device:R_Small R4
+U 1 1 61225B35
+P 10400 10300
+F 0 "R4" V 10204 10300 50  0000 C CNN
+F 1 "56" V 10295 10300 50  0000 C CNN
+F 2 "Resistor_SMD:R_0805_2012Metric_Pad1.20x1.40mm_HandSolder" H 10400 10300 50  0001 C CNN
+F 3 "~" H 10400 10300 50  0001 C CNN
+	1    10400 10300
+	0    1    1    0
+$EndComp
+$Comp
+L Device:R_Small R5
+U 1 1 612261DB
+P 10600 10500
+F 0 "R5" V 10404 10500 50  0000 C CNN
+F 1 "100" V 10495 10500 50  0000 C CNN
+F 2 "Resistor_SMD:R_0805_2012Metric_Pad1.20x1.40mm_HandSolder" H 10600 10500 50  0001 C CNN
+F 3 "~" H 10600 10500 50  0001 C CNN
+	1    10600 10500
+	0    1    1    0
+$EndComp
+Wire Wire Line
+	10300 10100 10750 10100
+Wire Wire Line
+	11250 10300 10500 10300
+Wire Wire Line
+	10300 10300 10100 10300
+Wire Wire Line
+	10100 10500 10500 10500
+Wire Wire Line
+	10700 10500 11750 10500
 $EndSCHEMATC

Commit message: Finish led magic
Parts:
- D4: footprint (none) -> LED_SMD:LED_LiteOn_LTST-C19HE1WT; symbol Device:LED_GABR -> Device:LED_RGBA; mouser 859-LTST-S310F2KT -> 859-LTST-C19HE1WT
- R3, R4: value 56 -> 15
- R5: value 100 -> 43
Connections:
- net +3V3: now also D4.4 (A); no longer D4.2 (A)
- net at D4.1 (RK): now also R5.2; no longer R4.2
- new net: D4.2 (GK), R4.2
Other:
- note added: "R VF=1.8-2.4 FC=30\nG VF=2.8-3.9 FC=20\nB VF=2.8-3.9 FC=20\nSupply=3.3"
Changed lines of the file:
@@
 $EndComp
 $Comp
-L Device:LED_GABR D4
+L Device:LED_RGBA D4
 U 1 1 5F871F9B
 P 9900 10300
 F 0 "D4" H 9900 10797 50  0000 C CNN
 F 1 "LED_GCBR_1" H 9900 10706 50  0000 C CNN
-F 2 "" H 9900 10250 50  0001 C CNN
+F 2 "LED_SMD:LED_LiteOn_LTST-C19HE1WT" H 9900 10250 50  0001 C CNN
 F 3 "~" H 9900 10250 50  0001 C CNN
-F 4 "859-LTST-S310F2KT" H 9900 10300 50  0001 C CNN "mouser"
+F 4 "859-LTST-C19HE1WT" H 9900 10300 50  0001 C CNN "mouser"
 	1    9900 10300
 	-1   0    0    1
@@
 P 10200 10100
 F 0 "R3" V 10004 10100 50  0000 C CNN
-F 1 "56" V 10095 10100 50  0000 C CNN
+F 1 "15" V 10095 10100 50  0000 C CNN
 F 2 "Resistor_SMD:R_0805_2012Metric_Pad1.20x1.40mm_HandSolder" H 10200 10100 50  0001 C CNN
 F 3 "~" H 10200 10100 50  0001 C CNN
@@
 P 10400 10300
 F 0 "R4" V 10204 10300 50  0000 C CNN
-F 1 "56" V 10295 10300 50  0000 C CNN
+F 1 "15" V 10295 10300 50  0000 C CNN
 F 2 "Resistor_SMD:R_0805_2012Metric_Pad1.20x1.40mm_HandSolder" H 10400 10300 50  0001 C CNN
 F 3 "~" H 10400 10300 50  0001 C CNN
@@
 P 10600 10500
 F 0 "R5" V 10404 10500 50  0000 C CNN
-F 1 "100" V 10495 10500 50  0000 C CNN
+F 1 "43" V 10495 10500 50  0000 C CNN
 F 2 "Resistor_SMD:R_0805_2012Metric_Pad1.20x1.40mm_HandSolder" H 10600 10500 50  0001 C CNN
 F 3 "~" H 10600 10500 50  0001 C CNN
@@
 Wire Wire Line
 	10700 10500 11750 10500
+Text Notes 10550 10900 0    39   ~ 0
+R VF=1.8-2.4 FC=30\nG VF=2.8-3.9 FC=20\nB VF=2.8-3.9 FC=20\nSupply=3.3
 $EndSCHEMATC

Commit message: sd card mouser pn
Parts:
- J3: mouser (none) -> 710-693072010801
Changed lines of the file:
@@
 F 2 "Connector_Card:microSD_HC_Wuerth_693072010801" H 3000 6400 50  0001 C CNN
 F 3 "http://katalog.we-online.de/em/datasheet/693072010801.pdf" H 1850 6100 50  0001 C CNN
+F 4 "710-693072010801" H 1850 6100 50  0001 C CNN "mouser"
 	1    1850 6100
 	-1   0    0    1
